Commit message: launch file works i think, need to write a simple client to test actions

File: models/arov_model.urdf (robot description, URDF)
Before this commit: robot AROV, 2 links, 1 joints
Joints:
- joint arov/base_joint: child  -> arov/base_footprint; parent  -> arov/base_link

File: models/asv_model.urdf (robot description, URDF)
Before this commit: robot ASV, 2 links, 1 joints
Joints:
- joint asv/base_joint: child  -> asv/base_footprint; parent  -> asv/base_link
